File: kicad_project/Heatbed-MK52.kicad_pcb (KiCad board)
At the start: 2 copper layers, 304 x 351 mm, 27 parts

Commit message: Add files via upload
Modified to make room for PCB cutting as it was too close to pads.
Routing:
- net Net-(D1-Pad1): track 49250.1 -> 49094.6 mm
